File: voltage-and-current-measurement.kicad_sch (KiCad schematic)
At the start: 27 parts

Commit message: Sch Voltage and current measurement
Parts:
- removed C? (x3): C_100n_0402, antmicro-footprints:C_0402_1005Metric, symbol antmicroCapacitors0402:C_100n_0402
- added C? (x7): C_100n_0402, antmicro-footprints:C_0402_1005Metric, symbol antmicroCapacitors0402:C_100n_0402
- added C?: C_1u_0402, antmicro-footprints:C_0402_1005Metric, symbol antmicroCapacitors0402:C_1u_0402
- added D? (x3): PESD5V0S2BQA, antmicro-footprints:TPD2E009DRTR, symbol antmicroTVSDiodes:PESD5V0S2BQA
- added FB?: FB_600Z_0.5A_Murata-BLM18AG_0603, antmicro-footprints:FB_0603_1608Metric, symbol antmicroFerriteBeadsandChips:FB_600Z_0.5A_Murata-BLM18AG_0603
- added R? (x7): R_15k4_0.1%_0402, antmicro-footprints:0402-res, symbol antmicroResistors0402:R_15k4_0.1%_0402
- added R? (x11): R_0R_0402, antmicro-footprints:R_0402_1005Metric, symbol antmicroResistors0402:R_0R_0402
- added R? (x7): R_100k_0.1%_0402, antmicro-footprints:0402-res, symbol antmicroResistors0402:R_100k_0.1%_0402
- added TP? (x11): TP_1mm_SMD, antmicro-footprints:TP_SMD_1mm, symbol antmicroTestPoints:TP_1mm_SMD
- added U? (x3): TMCS1100A2-Q1, gpu-cluster-backplane-footprints:SOIC-8_W3.9mm, symbol gpu-cluster-backplane:TMCS1100A2-Q1
- added U?: ADS7828, gpu-cluster-backplane-footprints:TSSOP-16_4.4x5mm_P0.65mm, symbol gpu-cluster-backplane:ADS7828
Connections:
- net VCC12V0 is gone; now on net LOAD_1: R?.2
- net C_ADC1: now also U?.1 (CH0); no longer U?.5 (CH4)
- net C_ADC2: now also U?.2 (CH1); no longer U?.4 (CH3)
- net C_ADC4: now also U?.4 (CH3); no longer U?.2 (CH1)
- net C_ADC5: now also U?.5 (CH4); no longer U?.1 (CH0)
- net GND: now also C?.2, C?.2, C?.2, C?.2, C?.2, C?.2, C?.2, C?.2, D?.3 (GND), D?.3 (GND), D?.3 (GND), R?.2, R?.2, R?.2, R?.2, R?.2, R?.2, R?.2, R?.2, R?.2, U?.11 (COM), U?.5 (GND), U?.5 (GND), U?.5 (GND), U?.6 (Vref), U?.6 (Vref), U?.6 (Vref), U?.9 (GND)
- net LOAD_2: now also R?.2
- net LOAD_3: now also R?.2
- net LOAD_4: now also R?.2
- net LOAD_5: now also R?.2
- net SCL: now also U?.14 (SCL)
- net SDA: now also U?.15 (SDA)
- net VCC3V3: now also C?.1, C?.1, C?.1, C?.1, C?.1, C?.1, C?.1, FB?.2, R?.1, R?.1, U?.16 (VDD), U?.8 (Vcc), U?.8 (Vcc), U?.8 (Vcc)
- net V_ADC1: now also TP?.1, U?.1 (CH0); no longer U?.8 (CH7)
- net V_ADC2: now reaches D?.2 (IO2)
- net V_ADC2: now also R?.2, TP?.1, U?.2 (CH1)
- net C_ADC6: now reaches U?.6 (CH5)
- net C_ADC6: now also TP?.1, U?.7 (Vout)
- net C_ADC7: now reaches U?.7 (CH6)
- net C_ADC7: now also TP?.1, U?.7 (Vout)
- new net: R?.1, R?.1, R?.1 (x7)
- new net: C?.1, FB?.1, U?.10 (REF)
- new net: R?.1, R?.2, U?.12 (A0)
- new net: R?.1, R?.2, U?.13 (A1)
- new net C_ADC8: TP?.1, U?.7 (Vout), U?.8 (CH7)
- new net C_MEAS_6: U?.1 (IN+), U?.2 (IN+)
- new net C_MEAS_7: U?.1 (IN+), U?.2 (IN+)
- new net C_MEAS_8: U?.1 (IN+), U?.2 (IN+)
- new net LOAD_6: R?.2, U?.3 (IN-), U?.4 (IN-)
- new net LOAD_7: R?.2, U?.3 (IN-), U?.4 (IN-)
- new net LOAD_8: R?.2, U?.3 (IN-), U?.4 (IN-)
- new net V_ADC3: D?.1 (IO1), R?.2, TP?.1, U?.3 (CH2)
- new net V_ADC4: D?.2 (IO2), R?.2, TP?.1, U?.4 (CH3)
- new net V_ADC5: D?.1 (IO1), R?.2, TP?.1, U?.5 (CH4)
- new net V_ADC6: D?.2 (IO2), R?.2, TP?.1, U?.6 (CH5)
- new net V_ADC7: D?.1 (IO1), R?.2, TP?.1, U?.7 (CH6)
- new net V_ADC8: D?.2 (IO2), R?.2, TP?.1, U?.8 (CH7)
- no-connect marks 3 -> 0
Other:
- note added: "ADC for current measurement"
- note added: "ADC for voltage measurement"
- note added: "Current measurement ADC inputs TPs"
- note added: "I2C adress: 0x48"
- note added: "I2C adress: 0x49"
- note added: "Remarks: LOAD_x signal should be separate track to measure voltage at connector"
- note added: "Voltage Measurement"
- note added: "Voltage measurement ADC inputs TPs"
- note removed: "ADC"
- note removed: "ADC inputs TPs"
- note removed: "Power filtration"
- note removed: "Sensors"
- note removed: "Supply"
- moved on the sheet: C?, D?, FB?, R?, TP?, U?

Commit message: WIP Sch components standarization
Parts:
- added C?: C_100n_0402, antmicro-footprints:C_0402_1005Metric, symbol antmicroCapacitors0402:C_100n_0402
- added FB?: FB_600Z_0.5A_Murata-BLM18AG_0603, antmicro-footprints:FB_0603_1608Metric, symbol antmicroFerriteBeadsandChips:FB_600Z_0.5A_Murata-BLM18AG_0603
- added R? (x4): R_0R_0402, antmicro-footprints:R_0402_1005Metric, symbol antmicroResistors0402:R_0R_0402
- added U?: ADS7828, antmicro-footprints:TSSOP-16_4.4x5mm_P0.65mm, symbol antmicroDataAcquisitionAnalogtoDigitalConvertersADC:ADS7828
Connections:
- net GND: now also C?.2, R?.2, R?.2
- net SCL: now also U?.14 (SCL)
- net SDA: now also U?.15 (SDA)
- net VCC3V3: now also FB?.2, R?.1, R?.1
- new net: R?.1, R?.2, U?.12 (A0)
- new net: R?.1, R?.2, U?.13 (A1)
- new net: C?.1, FB?.1, U?.10 (REF)

Commit message: WIP Standarization
Parts:
- removed C? (x2): C_100n_0402, antmicro-footprints:C_0402_1005Metric, symbol antmicroCapacitors0402:C_100n_0402
- removed FB? (x2): FB_600Z_0.5A_Murata-BLM18AG_0603, antmicro-footprints:FB_0603_1608Metric, symbol antmicroFerriteBeadsandChips:FB_600Z_0.5A_Murata-BLM18AG_0603
- removed R? (x8): R_0R_0402, antmicro-footprints:R_0402_1005Metric, symbol antmicroResistors0402:R_0R_0402
- removed U? (x2): ADS7828, gpu-cluster-backplane-footprints:TSSOP-16_4.4x5mm_P0.65mm, symbol gpu-cluster-backplane:ADS7828
- added C?: C_100n_0402, antmicro-footprints:C_0402_1005Metric, symbol antmicroCapacitors0402:C_100n_0402
- added FB?: FB_600Z_0.5A_Murata-BLM18AG_0603, antmicro-footprints:FB_0603_1608Metric, symbol antmicroFerriteBeadsandChips:FB_600Z_0.5A_Murata-BLM18AG_0603
- added R? (x4): R_0R_0402, antmicro-footprints:R_0402_1005Metric, symbol antmicroResistors0402:R_0R_0402
- added U?: ADS7828, antmicro-footprints:TSSOP-16_4.4x5mm_P0.65mm, symbol antmicroDataAcquisitionAnalogtoDigitalConvertersADC:ADS7828
Connections:
- net C_ADC1: now also U?.1 (CH0)
- net C_ADC2: now also U?.2 (CH1)
- net C_ADC3: now also U?.3 (CH2)
- net C_ADC4: now also U?.4 (CH3)
- net C_ADC5: now also U?.5 (CH4)
- net C_ADC6: now also U?.6 (CH5)
- net C_ADC7: now also U?.7 (CH6)
- net C_ADC8: now also U?.8 (CH7)
- net GND: now also U?.11 (COM), U?.9 (GND), C?.2, R?.2, R?.2, U?.11 (COM), U?.9 (GND)
- net SCL: now also U?.14 (SCL)
- net SDA: now also U?.15 (SDA)
- net VCC3V3: now also U?.16 (VDD), FB?.2, R?.1, R?.1, U?.16 (VDD)
- net V_ADC1: now also U?.1 (CH0)
- net V_ADC2: now also U?.2 (CH1)
- net V_ADC3: now also U?.3 (CH2)
- net V_ADC4: now also U?.4 (CH3)
- net V_ADC5: now also U?.5 (CH4)
- net V_ADC6: now also U?.6 (CH5)
- net V_ADC7: now also U?.7 (CH6)
- net V_ADC8: now also U?.8 (CH7)
- new net: R?.1, R?.2, U?.12 (A0)
- new net: R?.1, R?.2, U?.13 (A1)
- new net: C?.1, FB?.1, U?.10 (REF)
Other:
- moved on the sheet: C?, FB?, R?, TP?, U?
