File: fans-control.kicad_sch (KiCad schematic)
At the start: 53 parts, among them J2 PinHeader_1x4_P2.5mm_Drill1mm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, J3 PinHeader_1x4_P2.5mm_Drill1mm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, J4 PinHeader_1x4_P2.5mm_Drill1mm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, J5 PinHeader_1x4_P2.5mm_Drill1mm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, Q2 2N7002K-T1-E3, Q3 BSS138PW, U5 LM339_TSSOP_Split, U6 TS5A3359_VSSOP, U7 74CBTLV3257_VQFN, U8 74VHC153FT

Commit message: Cleanup project
Parts:
- gave numbers to parts that had none: 8
Changed lines of the file:
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@@
   (symbol (lib_id "antmicroFerriteBeadsandChips:FB_120Z_3A_Murata-BLM18SG_0603") (at 373.38 147.32 0) (unit 1)
     (in_bom yes) (on_board yes) (fields_autoplaced)
-    (property "Reference" "FB?" (id 0) (at 375.8819 140.97 0)
+    (property "Reference" "FB6" (id 0) (at 375.8819 140.97 0)
       (effects (font (size 1.27 1.27) (thickness 0.15)))
     )
@@
   (symbol (lib_name "1N4148WS-7-F_1") (lib_id "antmicroDiodesRectifiersSingle:1N4148WS-7-F") (at 360.68 189.23 90) (unit 1)
     (in_bom yes) (on_board yes) (fields_autoplaced)
-    (property "Reference" "D?" (id 0) (at 363.22 185.4199 90)
+    (property "Reference" "D9" (id 0) (at 363.22 185.4199 90)
       (effects (font (size 1.27 1.27) (thickness 0.15)) (justify right))
     )
@@
   (symbol (lib_name "1N4148WS-7-F_1") (lib_id "antmicroDiodesRectifiersSingle:1N4148WS-7-F") (at 359.41 156.21 90) (unit 1)
     (in_bom yes) (on_board yes) (fields_autoplaced)
-    (property "Reference" "D?" (id 0) (at 361.95 152.3999 90)
+    (property "Reference" "D7" (id 0) (at 361.95 152.3999 90)
       (effects (font (size 1.27 1.27) (thickness 0.15)) (justify right))
     )
@@
   (symbol (lib_name "1N4148WS-7-F_1") (lib_id "antmicroDiodesRectifiersSingle:1N4148WS-7-F") (at 360.68 86.36 90) (unit 1)
     (in_bom yes) (on_board yes) (fields_autoplaced)
-    (property "Reference" "D?" (id 0) (at 363.22 82.5499 90)
+    (property "Reference" "D8" (id 0) (at 363.22 82.5499 90)
       (effects (font (size 1.27 1.27) (thickness 0.15)) (justify right))
     )
@@
   (symbol (lib_name "1N4148WS-7-F_1") (lib_id "antmicroDiodesRectifiersSingle:1N4148WS-7-F") (at 359.41 123.19 90) (unit 1)
     (in_bom yes) (on_board yes) (fields_autoplaced)
-    (property "Reference" "D?" (id 0) (at 361.95 119.3799 90)
+    (property "Reference" "D6" (id 0) (at 361.95 119.3799 90)
       (effects (font (size 1.27 1.27) (thickness 0.15)) (justify right))
     )
@@
   (symbol (lib_id "antmicroFerriteBeadsandChips:FB_120Z_3A_Murata-BLM18SG_0603") (at 374.65 180.34 0) (unit 1)
     (in_bom yes) (on_board yes) (fields_autoplaced)
-    (property "Reference" "FB?" (id 0) (at 377.1519 173.99 0)
+    (property "Reference" "FB8" (id 0) (at 377.1519 173.99 0)
       (effects (font (size 1.27 1.27) (thickness 0.15)))
     )
@@
   (symbol (lib_id "antmicroFerriteBeadsandChips:FB_120Z_3A_Murata-BLM18SG_0603") (at 373.38 114.3 0) (unit 1)
     (in_bom yes) (on_board yes) (fields_autoplaced)
-    (property "Reference" "FB?" (id 0) (at 375.8819 107.95 0)
+    (property "Reference" "FB5" (id 0) (at 375.8819 107.95 0)
       (effects (font (size 1.27 1.27) (thickness 0.15)))
     )
@@
   (symbol (lib_id "antmicroFerriteBeadsandChips:FB_120Z_3A_Murata-BLM18SG_0603") (at 374.65 77.47 0) (unit 1)
     (in_bom yes) (on_board yes) (fields_autoplaced)
-    (property "Reference" "FB?" (id 0) (at 377.1519 71.12 0)
-      (effects (font (size 1.27 1.27) (thickness 0.15)))
-    )
+    (property "Reference" "FB7" (id 0) (at 377.1519 71.12 0)
+      (effects (font (size 1.27 1.27) (thickness 0.15)))
+    )

Commit message: Next batch of standardization
Parts:
- renumbered Q2 to Q4, Q3 to Q5
Changed lines of the file:
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@@
   (symbol (lib_id "antmicroTransistorsFETsMOSFETsSingle:2N7002K-T1-E3") (at 171.45 13.97 270) (unit 1)
     (in_bom yes) (on_board yes) (fields_autoplaced)
-    (property "Reference" "Q2" (id 0) (at 171.45 18.1337 90)
+    (property "Reference" "Q4" (id 0) (at 171.45 18.1337 90)
       (effects (font (size 1.524 1.524)))
     )
@@
   (symbol (lib_id "antmicroTransistorsFETsMOSFETsSingle:BSS138PW") (at 191.77 71.12 0) (unit 1)
     (in_bom yes) (on_board yes) (fields_autoplaced)
-    (property "Reference" "Q3" (id 0) (at 203.2 67.3099 0)
+    (property "Reference" "Q5" (id 0) (at 203.2 67.3099 0)
       (effects (font (size 1.27 1.27) (thickness 0.15)) (justify left))
     )
