File: power.kicad_sch (KiCad schematic)
At the start: 21 parts, among them U1 AP62301_TSOT, U3 AP62301_TSOT

Commit message: [#62160] Change ftdi-module.kicad_sch to power.kicad_sch
Other:
- moved on the sheet: C1, C10, C11, C14, C21, C22, C23, C5, D2, FB3, FB4, L1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
